File: Hardware/openbook_pcb.brd (EAGLE design)
At the start: 170.2 x 111.2 mm, 103 parts, among them IC1 BD5229G-TR, IC4 XC6220A331MR-G, J1 FH34SRJ-24S-0.5SH_99_, J2 SAMACSYS_PARTS_USB4110-GF-A, J3 QWIIC_RIGHT_ANGLE, J4 112A-TAAR-R03_ATTEND, Q1 20V/4.2A/52mΩ/1.4W, Q2 20V/4.2A/52mΩ/1.4W, Q3 SI1308EDL-T1-GE3, U1 W25Q512JVEIQ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

Commit message: fixed pcb issues
Parts:
- moved TP2 14.0 mm to (2.54, 72.4)
- moved TP1 11.4 mm to (2.48, 76.2)
- moved TP8 9.67 mm to (5.08, 36.8)
- moved TP10 8.13 mm to (95.2, 6.35)
- moved TP9 7.73 mm to (5.08, 31.8)
- moved TP4 6.84 mm to (71.1, 3.81)
- moved TP11 5.24 mm to (95.2, 2.54)
- moved TP12 4.02 mm to (95.2, 10.2)
- moved TP6 3.81 mm to (2.54, 68.6)
- moved TP16 3.81 mm to (5.08, 41.9)
- moved TP17 2.54 mm to (73.7, 35.6)
- moved C7 1.27 mm to (80.0, 26.7)
Routing:
- net RX: track 7.31 -> 28.5 mm
- net 3V3: track 521.0 -> 534.3 mm
- net MISO: track 75.7 -> 85.7 mm
- net SCK: track 166.5 -> 176.3 mm
- net TX: track 6.27 -> 15.4 mm
- net EPD_BUSY: track 126.8 -> 135.8 mm
- net EPD_3V3: track 38.6 -> 44.8 mm
- net EPD_DC: track 121.4 -> 126.1 mm
- net GND: track 714.9 -> 718.5 mm
- net EPD_CS: track 106.7 -> 110.3 mm
- net EPD_RST: track 137.9 -> 140.5 mm
- net SS_SD: track 94.1 -> 96.3 mm
- net N$3: track 11.0 -> 13.2 mm
- net N$1: track 18.1 -> 19.0 mm
